File: PIC24FJ64GA004 Dev Board/PIC24FJ64GA004 Dev Board.kicad_pcb (KiCad board)
At the start: 2 copper layers, 11 parts, among them U1 PIC24FJ64GA004-I_PT, U2 FT232RL, U3 XC6206PxxxMR

Commit message: added more
Parts:
- removed U1: PIC24FJ64GA004-I_PT, Package_QFP:TQFP-44_10x10mm_P0.8mm
- added C2: 0.1uf, Capacitor_SMD:C_0603_1608Metric, F.Cu at (142.5, 98.3)
- added C3: 0.1uf, Capacitor_SMD:C_0603_1608Metric, F.Cu at (142.5, 100.0)
- added C4: 0.1uf, Capacitor_SMD:C_0603_1608Metric, F.Cu at (142.5, 101.8)
- added C5: 0.1uf, Capacitor_SMD:C_0603_1608Metric, F.Cu at (142.5, 103.5)
- added C6: 0.1uf, Capacitor_SMD:C_0603_1608Metric, F.Cu at (145.0, 96.5)
- added C7: 0.1uf, Capacitor_SMD:C_0603_1608Metric, F.Cu at (145.0, 98.3)
- added C8: 0.1uf, Capacitor_SMD:C_0603_1608Metric, F.Cu at (145.0, 100.0)
- added C9: 0.1uf, Capacitor_SMD:C_0603_1608Metric, F.Cu at (145.0, 101.8)
- added J1: USB_C_Receptacle_USB2.0, Connector_USB:USB_C_Receptacle_GCT_USB4125-xx-x-0190_6P_TopMnt_Horizontal, F.Cu at (99.7, 62.2)
- added J2: Conn_01x22_Pin, Connector_PinHeader_2.54mm:PinHeader_1x22_P2.54mm_Vertical, B.Cu at (88.3, 59.1)
- added J3: Conn_01x22_Pin, Connector_PinHeader_2.54mm:PinHeader_1x22_P2.54mm_Vertical, B.Cu at (110.5, 59.1)
- added J4: Conn_PIC_ICSP_ICD, Connector_PinHeader_2.54mm:PinHeader_1x05_P2.54mm_Vertical_SMD_Pin1Left, F.Cu at (100.1, 111.6)
- added R6: 10k, Resistor_SMD:R_0603_1608Metric, F.Cu at (149.9, 100.2)
- added R7: 10k, Resistor_SMD:R_0603_1608Metric, F.Cu at (149.9, 101.9)
- added SW1: SW_Push, Button_Switch_SMD:SW_Push_1P1T_NO_6x6mm_H9.5mm, F.Cu at (144.0, 113.4)
- added U4: PIC24FJ64GA004-I_PT, Package_QFP:LQFP-44_10x10mm_P0.8mm, F.Cu at (99.5, 86.8)
- C1: footprint Capacitor_SMD:C_0201_0603Metric -> Capacitor_SMD:C_0603_1608Metric
- D1, D2: footprint LED_SMD:LED_0201_0603Metric -> LED_SMD:LED_0603_1608Metric
- R1, R2, R3, R4, R5: footprint Resistor_SMD:R_0201_0603Metric -> Resistor_SMD:R_0603_1608Metric
- U2: moved to B.Cu
- moved U2 177.3 mm to (161.3, 88.9), turned to 180 degrees
- moved R1 167.8 mm to (145.0, 103.5)
- moved D1 166.7 mm to (150.1, 96.5)
- moved D2 166.7 mm to (150.1, 98.3)
- moved R2 164.7 mm to (147.4, 96.5)
- moved R3 164.7 mm to (147.4, 98.3)
- moved R4 164.7 mm to (147.4, 100.0)
- moved R5 164.7 mm to (147.4, 101.8)
- moved C1 162.7 mm to (142.5, 96.5)
- moved U3 161.7 mm to (143.9, 106.6)
Connections:
- U2 pad 1: unconnected-(U2-TXD-Pad1) -> RX
- U2 pad 2: unconnected-(U2-DTR-Pad2) -> Net-(U2-DTR)
- U2 pad 5: unconnected-(U2-RXD-Pad5) -> TX
Routing:
- added copper zone on F.Cu, net GND
Other:
- board outline added: 27.4 x 59.1 mm
