File: PIC24FJ64GA004 Dev Board/_autosave-PIC24FJ64GA004 Dev Board.kicad_pcb (KiCad board)
At the start: 2 copper layers, 24.4 x 57.5 mm, 29 parts, among them J1 USB_C_Receptacle_USB2.0, J2 Conn_01x22_Pin, J3 Conn_01x22_Pin, J4 Conn_PIC_ICSP_ICD, SW1 SW_Push, U2 FT232RL, U3 XC6206PxxxMR, U4 PIC24FJ64GA004-I_PT, Y1 Crystal

Commit message: g
Routing:
- net PGC2: track 51.2 -> 47.5 mm, vias 0 -> 1
- net PGD2: track 44.6 -> 41.6 mm, vias 0 -> 1
- net P5: track 18.5 -> 17.3 mm
- net P4: track 21.0 -> 19.9 mm
- net GND: track 105.7 -> 104.7 mm, vias 34 -> 36
- net +3V3: track 176.0 -> 175.0 mm
- net P3: track 23.1 -> 22.4 mm
Other:
- board size 24.4 x 57.5 mm -> 23.9 x 57.3 mm
