File: PIC24FJ64GA004 Dev Board/_autosave-PIC24FJ64GA004 Dev Board.kicad_sch (KiCad schematic)
At the start: 29 parts, among them J1 USB_C_Receptacle_USB2.0, J2 Conn_01x22_Pin, J3 Conn_01x22_Pin, J4 Conn_PIC_ICSP_ICD, SW1 SW_Push, U2 FT232RL, U3 XC6206PxxxMR, U4 PIC24FJ64GA004-I_PT, Y1 Crystal

Commit message: g
Parts:
- C2: value 0.1uf -> 4.7uf
- R7: value 10k -> 1k
Connections:
- net MCLR: no longer J4.1 (~{MCLR}/VPP)
- net MCLRI: now reaches C5.1, R6.2, R7.1, SW1.2
- net MCLRI: now also J4.1 (~{MCLR}/VPP)
Other:
- moved on the sheet: R7
Changed lines of the file:
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@@
+    (stroke (width 0) (type default))
+  )
+  (wire (pts (xy 273.05 104.14) (xy 270.51 104.14))
     (stroke (width 0) (type default))
   )
@@
     (stroke (width 0) (type default))
   )
-  (wire (pts (xy 250.19 104.14) (xy 255.27 104.14))
+  (wire (pts (xy 250.19 104.14) (xy 262.89 104.14))
     (stroke (width 0) (type default))
   )
@@
     (stroke (width 0) (type default))
   )
+  (wire (pts (xy 52.07 118.11) (xy 48.26 118.11))
+    (stroke (width 0) (type default))
+  )
   (wire (pts (xy 217.17 125.73) (xy 217.17 128.27))
     (stroke (width 0) (type default))
@@
     )
   )
+  (global_label "MCLRI" (shape input) (at 260.35 104.14 90) (fields_autoplaced)
+    (effects (font (size 1.27 1.27)) (justify left))
+    (property "Intersheetrefs" "${INTERSHEET_REFS}" (at 260.35 95.5305 90)
+      (effects (font (size 1.27 1.27)) (justify left) hide)
+    )
+  )
   (global_label "P25" (shape input) (at 168.91 95.25 0) (fields_autoplaced)
     (effects (font (size 1.27 1.27)) (justify left))
@@
     )
   )
-  (global_label "MCLR" (shape input) (at 48.26 118.11 0) (fields_autoplaced)
-    (effects (font (size 1.27 1.27)) (justify left))
-    (property "Intersheetrefs" "${INTERSHEET_REFS}" (at 56.2647 118.11 0)
+  (global_label "MCLRI" (shape input) (at 52.07 118.11 0) (fields_autoplaced)
+    (effects (font (size 1.27 1.27)) (justify left))
+    (property "Intersheetrefs" "${INTERSHEET_REFS}" (at 60.6795 118.11 0)
       (effects (font (size 1.27 1.27)) (justify left) hide)
     )
@@
     )
   )
-  (global_label "MCLR" (shape input) (at 262.89 104.14 0) (fields_autoplaced)
-    (effects (font (size 1.27 1.27)) (justify left))
-    (property "Intersheetrefs" "${INTERSHEET_REFS}" (at 270.8947 104.14 0)
+  (global_label "MCLR" (shape input) (at 273.05 104.14 0) (fields_autoplaced)
+    (effects (font (size 1.27 1.27)) (justify left))
+    (property "Intersheetrefs" "${INTERSHEET_REFS}" (at 281.0547 104.14 0)
       (effects (font (size 1.27 1.27)) (justify left) hide)
     )
@@
       (effects (font (size 1.27 1.27)) (justify left))
     )
-    (property "Value" "0.1uf" (at 120.65 160.02 0)
+    (property "Value" "4.7uf" (at 120.65 160.02 0)
       (effects (font (size 1.27 1.27)) (justify left))
     )
@@
     )
   )
-  (symbol (lib_id "Device:R") (at 259.08 104.14 90) (unit 1)
-    (in_bom yes) (on_board yes) (dnp no) (fields_autoplaced)
-    (property "Reference" "R7" (at 259.08 97.79 90)
-      (effects (font (size 1.27 1.27)))
-    )
-    (property "Value" "10k" (at 259.08 100.33 90)
-      (effects (font (size 1.27 1.27)))
-    )
-    (property "Footprint" "Resistor_SMD:R_0603_1608Metric" (at 259.08 105.918 90)
-      (effects (font (size 1.27 1.27)) hide)
-    )
-    (property "Datasheet" "~" (at 259.08 104.14 0)
-      (effects (font (size 1.27 1.27)) hide)
-    )
+  (symbol (lib_id "Device:R") (at 266.7 104.14 90) (unit 1)
+    (in_bom yes) (on_board yes) (dnp no) (fields_autoplaced)
+    (property "Reference" "R7" (at 266.7 97.79 90)
+      (effects (font (size 1.27 1.27)))
+    )
+    (property "Value" "1k" (at 266.7 100.33 90)
+      (effects (font (size 1.27 1.27)))
+    )
+    (property "Footprint" "Resistor_SMD:R_0603_1608Metric" (at 266.7 105.918 90)
+      (effects (font (size 1.27 1.27)) hide)
+    )
+    (property "Datasheet" "~" (at 266.7 104.14 0)
+      (effects (font (size 1.27 1.27)) hide)
+    )
