File: devboard/PIC24FJ64GA004 Dev Board/PIC24FJ64GA004 Dev Board.kicad_pcb (KiCad board)
At the start: 2 copper layers, 23.9 x 57.3 mm, 39 parts, among them J1 USB_C_Receptacle_USB2.0, J2 Conn_01x22_Pin, J3 Conn_01x22_Pin, J4 Conn_PIC_ICSP_ICD, SW1 SW_Push, U1 23LC1024T-I/SN, U2 FT232RL, U3 XC6206PxxxMR, U4 PIC24FJ64GA004-I_PT, U5 25CSM04xxSN, U6 SST25VF080B-50-4x-S2Ax, Y1 Crystal_GND24

Commit message: gdfs
Parts:
- U1: footprint Package_SO:SOIC-8-N7_3.9x4.9mm_P1.27mm -> Package_SO:SOIC-8_3.9x4.9mm_P1.27mm
- renumbered RX to D1, TX to D2
Routing:
- net +3V3: track 224.2 -> 225.4 mm
