File: devboard/PIC24FJ64GA004 Dev Board/PIC24FJ64GA004 Dev Board.kicad_sch (KiCad schematic)
At the start: 38 parts, among them J1 USB_C_Receptacle_USB2.0, J2 Conn_01x22_Pin, J3 Conn_01x22_Pin, J4 Conn_PIC_ICSP_ICD, SW1 SW_Push, U2 FT232RL, U2 SST25VF080B-50-4x-S2Ax, U3 23LC1024T-I/SN, U3 XC6206PxxxMR, U4 PIC24FJ64GA004-I_PT, Y1 Crystal_GND24

Commit message: gdfs
Parts:
- U3: footprint Package_SO:SOIC-8-N7_3.9x4.9mm_P1.27mm -> Package_SO:SOIC-8_3.9x4.9mm_P1.27mm
Changed lines of the file:
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@@
       (effects (font (size 1.524 1.524)))
     )
-    (property "Footprint" "Package_SO:SOIC-8-N7_3.9x4.9mm_P1.27mm" (at 124.46 175.26 0)
+    (property "Footprint" "Package_SO:SOIC-8_3.9x4.9mm_P1.27mm" (at 124.46 175.26 0)
       (effects (font (size 1.27 1.27) italic) hide)
     )
